Commit message: Editing while debugging

File: aruco_model_generation/urdf/common/aruco_robot.urdf.xacro (robot description, xacro)
@@ -3,6 +3,9 @@
     <xacro:arg name="id" default="100"/>
     <name>aruco_$(arg id)</name>
-    <xacro:arg name="size" default="100"/>
+    <xacro:arg name="sizemm" default="100"/>
     <xacro:include filename="$(find aruco_model_generation)/urdf/common/base_aruco_panel.urdf.xacro"/>
-    <xacro:aruco_panel width="$(arg size)" thickness="0.001" id="$(arg id)"/>
+    <xacro:macro name="sized_panel" params="sizemm">
+        <xacro:aruco_panel width="${sizemm/1000.0}" thickness="0.001" id="$(arg id)"/>
+    </xacro:macro>
+    <xacro:sized_panel sizemm="$(arg sizemm)"/>
 </robot>

File: aruco_model_generation/urdf/common/base_aruco_panel.urdf.xacro (robot description, xacro)
@@ -21,5 +21,5 @@
         </script>
     </material>
-    <link name="base_link">
+    <link name="aruco_${id}_panel">
         <collision>
             <xacro:panel_box width="${width}" thickness="${thickness}"/>
@@ -38,5 +38,5 @@
         </inertial>
     </link>
-    <gazebo reference="base_link">
+    <gazebo reference="aruco_${id}_panel">
         <material>Aruco/Aruco${id}</material>
     </gazebo>
